File: surfacemount.brd (EAGLE design)
At the start: 79.2 x 33.6 mm, 5 parts, among them J1 2.1MMJACKTHM

Commit message: Fixed smd
Parts:
- LED1: value (none) -> Red
- U$1: value (none) -> 330Ohms
- moved J1 53.5 mm to (68.0, 57.0), turned to 90 degrees
- moved LED1 49.7 mm to (31.0, 60.0)
- moved S1 41.6 mm to (44.0, 48.0), turned to 180 degrees
- moved U$1 41.4 mm to (15.0, 52.0), turned to 270 degrees
Connections:
- net N$3: now also S1.2
- net N$4: now also S1.3
Routing:
- net N$1: track 0.00 -> 44.2 mm
- net N$3: track 0.00 -> 24.2 mm
- net N$4: track 0.00 -> 23.4 mm
- net N$2: track 0.00 -> 18.2 mm
Changed lines of the file:
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@@
 <elements>
 <element name="U$3" library="Logos-Large" package="UCSD_LOGO_LARGE" value="" x="3" y="58"/>
-<element name="J1" library="georgelachow-Lab2" package="PJ-102A" value="2.1MMJACKTHM" x="17" y="41"/>
-<element name="S1" library="georgelachow-Lab2" package="1301.9315" value="" x="10" y="24"/>
-<element name="LED1" library="georgelachow-Lab2" package="LED5MM" value="" x="6" y="17"/>
-<element name="U$1" library="georgelachow-Lab2" package="RESAD1160W55L680D260_HS" value="" x="9" y="11">
-<attribute name="VAL" value="" x="9" y="11" size="1.778" layer="27" display="off"/>
-<attribute name="PWR" value="" x="9" y="11" size="1.778" layer="27" display="off"/>
-<attribute name="CASE" value="" x="9" y="11" size="1.778" layer="27" display="off"/>
-<attribute name="TOL" value="" x="9" y="11" size="1.778" layer="27" display="off"/>
-<attribute name="URL" value="" x="9" y="11" size="1.778" layer="27" display="off"/>
-<attribute name="DIST1PN" value="" x="9" y="11" size="1.778" layer="27" display="off"/>
-<attribute name="DIST1" value="" x="9" y="11" size="1.778" layer="27" display="off"/>
-<attribute name="MFR" value="" x="9" y="11" size="1.778" layer="27" display="off"/>
-<attribute name="MPN" value="" x="9" y="11" size="1.778" layer="27" display="off"/>
-<attribute name="DESC" value="" x="9" y="11" size="1.778" layer="27" display="off"/>
-<attribute name="SIZE" value="" x="9" y="11" size="1.778" layer="27" display="off"/>
+<element name="S1" library="georgelachow-Lab2" package="1301.9315" value="" x="44" y="48" rot="R180"/>
+<element name="J1" library="georgelachow-Lab2" package="PJ-102A" value="2.1MMJACKTHM" x="68" y="57" rot="R90"/>
+<element name="LED1" library="georgelachow-Lab2" package="LED5MM" value="Red" x="31" y="60"/>
+<element name="U$1" library="georgelachow-Lab2" package="RESAD1160W55L680D260_HS" value="330Ohms" x="15" y="52" rot="R270">
+<attribute name="VAL" value="" x="15" y="52" size="1.778" layer="27" rot="R270" display="off"/>
+<attribute name="PWR" value="" x="15" y="52" size="1.778" layer="27" rot="R270" display="off"/>
+<attribute name="CASE" value="" x="15" y="52" size="1.778" layer="27" rot="R270" display="off"/>
+<attribute name="TOL" value="" x="15" y="52" size="1.778" layer="27" rot="R270" display="off"/>
+<attribute name="URL" value="" x="15" y="52" size="1.778" layer="27" rot="R270" display="off"/>
+<attribute name="DIST1PN" value="" x="15" y="52" size="1.778" layer="27" rot="R270" display="off"/>
+<attribute name="DIST1" value="" x="15" y="52" size="1.778" layer="27" rot="R270" display="off"/>
+<attribute name="MFR" value="" x="15" y="52" size="1.778" layer="27" rot="R270" display="off"/>
+<attribute name="MPN" value="" x="15" y="52" size="1.778" layer="27" rot="R270" display="off"/>
+<attribute name="DESC" value="" x="15" y="52" size="1.778" layer="27" rot="R270" display="off"/>
+<attribute name="SIZE" value="" x="15" y="52" size="1.778" layer="27" rot="R270" display="off"/>
 </element>
 </elements>
@@
 <contactref element="J1" pad="TIP"/>
 <contactref element="LED1" pad="A"/>
-<wire x1="4.73" y1="17" x2="16.13" y2="36.655" width="0" layer="19" extent="1-1"/>
+<wire x1="30.7848" y1="59.8932" x2="29.8704" y2="59.8932" width="0.1524" layer="16"/>
+<wire x1="34.4424" y1="56.2356" x2="30.7848" y2="59.8932" width="0.1524" layer="16"/>
+<wire x1="72.2376" y1="56.2356" x2="34.4424" y2="56.2356" width="0.1524" layer="16"/>
+<wire x1="29.8704" y1="59.8932" x2="29.73" y2="60" width="0.1524" layer="16"/>
+<wire x1="72.2376" y1="56.2356" x2="72.345" y2="56.13" width="0.1524" layer="16"/>
 </signal>
 <signal name="N$2">
 <contactref element="LED1" pad="K"/>
 <contactref element="U$1" pad="1"/>
-<wire x1="3.2" y1="11" x2="7.27" y2="17" width="0" layer="19" extent="1-1"/>
+<wire x1="30.1752" y1="57.912" x2="15.0876" y2="57.912" width="0.1524" layer="1"/>
+<wire x1="32.1564" y1="59.8932" x2="30.1752" y2="57.912" width="0.1524" layer="1"/>
+<wire x1="15.0876" y1="57.912" x2="15" y2="57.8" width="0.1524" layer="1"/>
+<wire x1="32.1564" y1="59.8932" x2="32.27" y2="60" width="0.1524" layer="1"/>
 </signal>
 <signal name="N$3">
 <contactref element="U$1" pad="2"/>
+<contactref element="S1" pad="2"/>
+<wire x1="15.3924" y1="45.8724" x2="38.862" y2="45.8724" width="0.1524" layer="1"/>
+<wire x1="15.0876" y1="46.1772" x2="15.3924" y2="45.8724" width="0.1524" layer="1"/>
+<wire x1="38.862" y1="45.8724" x2="39" y2="45.75" width="0.1524" layer="1"/>
+<wire x1="15.0876" y1="46.1772" x2="15" y2="46.2" width="0.1524" layer="1"/>
 </signal>
 <signal name="N$4">
+<contactref element="S1" pad="3"/>
 <contactref element="J1" pad="RING"/>
+<wire x1="72.2376" y1="50.292" x2="49.0728" y2="50.292" width="0.1524" layer="1"/>
+<wire x1="49.0728" y1="50.292" x2="49" y2="50.25" width="0.1524" layer="1"/>
+<wire x1="72.2376" y1="50.292" x2="72.345" y2="50.23" width="0.1524" layer="1"/>
 </signal>
 </signals>
