File: surfacemount.sch (EAGLE design)
At the start: 4 parts, among them J1 2.1MMJACKTHM

Commit message: Fixed smd
Parts:
- LED1: value (none) -> Red
- U$1: value (none) -> 330Ohms
Connections:
- net N$3: now also S1.2
- net N$4: now also S1.3
Other:
- moved on the sheet: J1, LED1, U$1
Changed lines of the file:
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@@
 </classes>
 <parts>
+<part name="S1" library="georgelachow-Lab2" deviceset="1301.9315" device=""/>
 <part name="J1" library="georgelachow-Lab2" deviceset="2.1MMJACK" device="THM"/>
-<part name="S1" library="georgelachow-Lab2" deviceset="1301.9315" device=""/>
-<part name="LED1" library="georgelachow-Lab2" deviceset="LED" device="5MM"/>
-<part name="U$1" library="georgelachow-Lab2" deviceset="RESISTOR" device="TH-1/4W-CARBON"/>
+<part name="LED1" library="georgelachow-Lab2" deviceset="LED" device="5MM" value="Red"/>
+<part name="U$1" library="georgelachow-Lab2" deviceset="RESISTOR" device="TH-1/4W-CARBON" value="330Ohms"/>
 </parts>
 <sheets>
@@
 </plain>
 <instances>
-<instance part="J1" gate="G$1" x="60.96" y="83.82"/>
-<instance part="S1" gate="G$1" x="78.74" y="76.2"/>
-<instance part="LED1" gate="G$1" x="68.58" y="96.52" rot="R90"/>
-<instance part="U$1" gate="G$1" x="81.28" y="96.52"/>
+<instance part="S1" gate="G$1" x="86.36" y="83.82"/>
+<instance part="J1" gate="G$1" x="66.04" y="83.82"/>
+<instance part="LED1" gate="G$1" x="73.66" y="96.52" rot="R90"/>
+<instance part="U$1" gate="G$1" x="86.36" y="96.52"/>
 </instances>
 <busses>
@@
 <pinref part="J1" gate="G$1" pin="TIP"/>
 <pinref part="LED1" gate="G$1" pin="A"/>
-<wire x1="66.04" y1="86.36" x2="66.04" y2="96.52" width="0.1524" layer="91"/>
+<wire x1="71.12" y1="86.36" x2="71.12" y2="96.52" width="0.1524" layer="91"/>
 </segment>
 </net>
@@
 <pinref part="LED1" gate="G$1" pin="C"/>
 <pinref part="U$1" gate="G$1" pin="1"/>
-<wire x1="73.66" y1="96.52" x2="76.2" y2="96.52" width="0.1524" layer="91"/>
+<wire x1="78.74" y1="96.52" x2="81.28" y2="96.52" width="0.1524" layer="91"/>
 </segment>
 </net>
@@
 <segment>
 <pinref part="U$1" gate="G$1" pin="2"/>
-<wire x1="86.36" y1="96.52" x2="86.36" y2="86.36" width="0.1524" layer="91"/>
-<wire x1="76.2" y1="86.36" x2="86.36" y2="86.36" width="0.1524" layer="91"/>
+<wire x1="91.44" y1="96.52" x2="91.44" y2="86.36" width="0.1524" layer="91"/>
+<pinref part="S1" gate="G$1" pin="2"/>
 </segment>
 </net>
 <net name="N$4" class="0">
 <segment>
+<pinref part="S1" gate="G$1" pin="3"/>
 <pinref part="J1" gate="G$1" pin="RING"/>
-<wire x1="76.2" y1="81.28" x2="66.04" y2="81.28" width="0.1524" layer="91"/>
+<wire x1="81.28" y1="81.28" x2="71.12" y2="81.28" width="0.1524" layer="91"/>
 </segment>
 </net>
